File: hardware/Template.kicad_sch (KiCad schematic)
At the start: 0 parts

Commit message: WIP: Support for GitLab
Other:
- title: Template -> (none)
Changed lines of the file:
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@@
 	(paper "A3")
 	(title_block
-		(title "Template")
+		(title "")
 		(date "2025-06-05")
 		(rev "${REVISION}")
